Commit message: xacro parser

File: data/sample.xacro (robot description, xacro)
@@ -1,4 +1,5 @@
 <robot xmlns:xacro="http://www.ros.org/wiki/xacro">
   <!-- Define a macro with parameters prefix, parent, and reflect - partially with default values -->
+  <xacro:property name="test" value="1"/>
   <xacro:macro name="arm" params="prefix:='' parent reflect:=1">
     <xacro:property name="prefix_" value='${prefix + "_" if prefix else ""}' />

Commit message: add lexer and eval

File: data/sample.xacro (robot description, xacro)
@@ -3,5 +3,5 @@
   <xacro:property name="test" value="1"/>
   <xacro:macro name="arm" params="prefix:='' parent reflect:=1">
-    <xacro:property name="prefix_" value='${prefix + "_" if prefix else ""}' />
+    <xacro:property name="prefix_" value='${prefix}_' />
     <upperarm prefix="${prefix}" reflect="${reflect}" parent="${parent}" />
     <forearm prefix="${prefix}" reflect="${reflect}" parent="${prefix_}elbow" />

Commit message: fix if/unless

File: data/sample.xacro (robot description, xacro)
@@ -1,9 +1,10 @@
 <robot xmlns:xacro="http://www.ros.org/wiki/xacro">
-  <!-- Define a macro with parameters prefix, parent, and reflect - partially with default values -->
-  <xacro:property name="test" value="1"/>
+  <xacro:property name="var" value="test"/>
   <xacro:macro name="arm" params="prefix:='' parent reflect:=1">
     <xacro:property name="prefix_" value='${prefix}_' />
     <upperarm prefix="${prefix}" reflect="${reflect}" parent="${parent}" />
-    <forearm prefix="${prefix}" reflect="${reflect}" parent="${prefix_}elbow" />
+    <xacro:if value="${var == 'test'}">
+      <forearm prefix="${prefix}" reflect="${reflect}" parent="${prefix_}elbow" />
+    </xacro:if>
   </xacro:macro>
   <!-- Instantiate the macro with different parameters -->
